File: E13.kicad_pcb (KiCad board)
At the start: 2 copper layers, 48.4 x 21.6 mm, 26 parts, among them J1 2x2 Connector, J2 WS-bus output, J3 WS-bus input, J4 UPDI, J5 Debug, J7 Screw Connector, U1 AVR-64da32, U2 MIC5205-5.0YM5

Commit message: initial
Parts:
- removed U1: AVR-64da32, Package_DFN_QFN:QFN-32-1EP_5x5mm_P0.5mm_EP3.1x3.1mm
- added C5: 100n, Capacitor_SMD:C_0603_1608Metric, F.Cu at (116.8, 88.7)
- added IC1: AVR64DB32-I_RXB, Package_DFN_QFN:QFN-32-1EP_5x5mm_P0.5mm_EP3.3x3.3mm, F.Cu at (120.6, 90.4)
- moved C3 0.47 mm to (123.9, 92.5)
- moved R15 0.09 mm to (113.8, 85.2)
- moved R16 0.07 mm to (116.4, 85.2)
Routing:
- net OUT4: track 27.3 -> 15.0 mm
- net OUT3: track 25.5 -> 16.5 mm
- net OUT2: track 29.3 -> 22.8 mm
- net DAC: track 0.00 -> 4.88 mm
- net OUT1: track 28.7 -> 24.0 mm
- net Net-(IC1-Pad6): track 3.83 -> 8.21 mm
- net GND: track 8.47 -> 5.70 mm, vias 8 -> 9
- net Net-(IC1-Pad7): track 2.28 -> 4.32 mm
- net Net-(IC1-Pad8): track 6.41 -> 8.17 mm
- net Net-(IC1-Pad12): track 19.6 -> 18.2 mm
- net Net-(IC1-Pad9): track 9.07 -> 9.71 mm
- net DI: vias 0 -> 1
Other:
- rule pad_to_mask_clearance: 0.051 -> 0
- rule trace_min: 0.15 -> 0.1
- rule via_min_size: 0.4 -> 0.3
- board text added: "E13.1"
- board text added: "FS 2024"
- board text removed: "E13.0"
- board text removed: "FS 2023"

Commit message: Initial commit
Parts:
- added RN1: 4x 22k, Resistor_SMD:R_Array_Convex_4x0603, F.Cu at (125.5, 87.9)
- C5: moved to B.Cu
- J1: value 2x2 Connector -> Multiplex out
- J5: value Debug -> Debug IF
- J7: value Screw Connector -> Multiplex out
- JP1: value SolderJumper_2_Open -> skip LDO
- moved C5 2.87 mm to (119.6, 87.9), turned to 315 degrees
- moved R16 2.73 mm to (118.9, 84.2)
- moved R17 2.61 mm to (116.4, 84.2)
- moved R14 0.99 mm to (111.3, 84.2)
- moved R15 0.97 mm to (113.8, 84.2)
Connections:
- IC1 pad 1: (no net) -> Net-(IC1-Pad1)
- IC1 pad 11: (no net) -> OUT1
- IC1 pad 13: (no net) -> OUT2
- IC1 pad 14: (no net) -> OUT3
- IC1 pad 15: (no net) -> OUT4
- IC1 pad 2: (no net) -> Net-(IC1-Pad2)
- IC1 pad 3: (no net) -> Net-(IC1-Pad3)
- IC1 pad 4: (no net) -> Net-(IC1-Pad4)
- R16 pad 2: OUT2 -> OUT1
- R17 pad 2: OUT1 -> OUT2
Routing:
- net OUT4: track 15.0 -> 43.9 mm, vias 0 -> 2
- net OUT3: track 16.5 -> 39.5 mm, vias 0 -> 2
- net OUT2: track 22.8 -> 41.5 mm, vias 0 -> 2
- net OUT1: track 24.0 -> 36.4 mm, vias 0 -> 2
- net Net-(IC1-Pad7): track 4.32 -> 8.38 mm, vias 0 -> 2
- net Net-(IC1-Pad1): track 0.00 -> 2.37 mm
- net Net-(IC1-Pad2): track 0.00 -> 2.24 mm
- net Net-(IC1-Pad3): track 0.00 -> 2.12 mm
- net Net-(IC1-Pad9): track 9.71 -> 11.8 mm, vias 0 -> 2
- net Net-(IC1-Pad4): track 0.00 -> 1.99 mm
- net Net-(IC1-Pad8): track 8.17 -> 9.85 mm, vias 0 -> 2
- net Net-(IC1-Pad6): track 8.21 -> 6.60 mm, vias 0 -> 2
- net Net-(IC1-Pad12): track 18.2 -> 17.6 mm
- net DAC: track 4.88 -> 4.95 mm, vias 0 -> 2
- net GND: vias 9 -> 8
Other:
- board text removed: "2"
- board text removed: "3"
