File: E13.kicad_pcb (KiCad board)
At the start: 2 copper layers, 48.4 x 21.6 mm, 28 parts, among them IC1 AVR64DB32-I_RXB, J1 Multiplex out, J2 WS-bus output, J3 WS-bus input, J4 UPDI, J5 Debug IF, J7 Multiplex out, U2 MIC5205-5.0YM5

Commit message: mod: documentation
Parts:
- R20: moved to F.Cu
- moved R20 3.04 mm to (117.6, 95.7), turned to 180 degrees
Routing:
- net VDD: track 18.0 -> 13.8 mm, vias 2 -> 1
- net Net-(D2-Pad2): track 0.00 -> 1.47 mm, vias 1 -> 0
